File: hardware/ControlsLeader_PCB/ControlsLeader_PCB.kicad_sch (KiCad schematic)
At the start: 20 parts, among them J1 CarCANConnector_Out, J12 SteeringConn_01x07, J15 IgnConn_01x04, J17 Conn_01x02, J2 PeripheralCAN_out, J3 CarCANConnector_In, J4 PeripheralCAN_in, J6 Conn_2Rows-13Pins, J8 Dash_Lsom_Horn_Lights_PWR, U2 LeaderSOM

Commit message: BOM!
Parts:
- D28, D30: P/N (none) -> LS Q976.01-N1Q2-1-20-R18
- D29: P/N (none) -> VSSAF522-M3/H
- F1: P/N (none) -> 3568
- J1, J3: P/N 1053091102 -> 1053131102
- J12: P/N (none) -> 1053131107
- J15: P/N (none) -> 1053131104
- J17: P/N (none) -> 1053131102
- J2, J4: P/N 105309-1204 -> 1053131104
- J6: P/N (none) -> 1053141112
- J8: P/N (none) -> 1053141106
- R10, R56: footprint Capacitor_SMD:C_0603_1608Metric_Pad1.08x0.95mm_HandSolder -> Resistor_SMD:R_0603_1608Metric_Pad0.98x0.95mm_HandSolder; P/N (none) -> CRCW12101K10FKEAHP
- U2: now left out of the parts list
Changed lines of the file:
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@@
 			)
 		)
-		(property "Description" "Generic connector, double row, 07 pins, odd/even pin numbering scheme (row 1 odd numbers, row 2 even numbers), script generated (kicad-library-utils/schlib/autogen/connector/)"
+		(property "Description" "PWR"
+			(at 93.98 39.37 0)
+			(effects
+				(font
+					(size 1.27 1.27)
+				)
+				(hide yes)
+			)
+		)
+		(property "P/N" "1053141106"
 			(at 93.98 39.37 0)
 			(effects
@@
 			)
 		)
-		(property "Description" "Generic connector, double row, 13 pins, odd/even pin numbering scheme (row 1 odd numbers, row 2 even numbers), script generated (kicad-library-utils/schlib/autogen/connector/)"
+		(property "Description" "Dash Conn"
+			(at 165.1 39.37 0)
+			(effects
+				(font
+					(size 1.27 1.27)
+				)
+				(hide yes)
+			)
+		)
+		(property "P/N" "1053141112"
 			(at 165.1 39.37 0)
 			(effects
@@
 			)
 		)
-		(property "Description" "Light emitting diode"
+		(property "Description" "3.3LDO LED"
 			(at 267.97 154.94 0)
 			(effects
@@
 			)
 		)
+		(property "P/N" "LS Q976.01-N1Q2-1-20-R18"
+			(at 267.97 154.94 0)
+			(effects
+				(font
+					(size 1.27 1.27)
+				)
+				(hide yes)
+			)
+		)
 		(pin "2"
 		)
@@
 			)
 		)
-		(property "Description" "75V 0.15A Fast switching Diode, SOD-523"
+		(property "Description" "Horn_Conn_Flyback"
 			(at 198.12 173.99 0)
 			(effects
@@
 		(property "Sim.Pins" "1=K 2=A"
 			(at 198.12 173.99 0)
+			(effects
+				(font
+					(size 1.27 1.27)
+				)
+				(hide yes)
+			)
+		)
+		(property "P/N" "VSSAF522-M3/H"
+			(at 198.12 173.99 90)
 			(effects
 				(font
@@
 			)
 		)
-		(property "Description" "Generic connector, single row, 01x02, script generated (kicad-library-utils/schlib/autogen/connector/)"
+		(property "Description" "Horn Conn"
+			(at 207.01 172.72 0)
+			(effects
+				(font
+					(size 1.27 1.27)
+				)
+				(hide yes)
+			)
+		)
+		(property "P/N" "1053131102"
 			(at 207.01 172.72 0)
 			(effects
@@
 			)
 		)
-		(property "Description" "Connection to the car's Peripheral CAN bus."
+		(property "Description" "PH Can In"
 			(at 146.05 168.91 0)
 			(effects
@@
 			)
 		)
-		(property "P/N" "105309-1204 "
+		(property "P/N" "1053131104"
 			(at 146.05 168.91 0)
 			(effects
@@
 			)
 		)
-		(property "Description" "Fuse"
+		(property "Description" "Fuse_3.3LDO"
 			(at 261.62 158.75 0)
+			(effects
+				(font
+					(size 1.27 1.27)
+				)
+				(hide yes)
+			)
+		)
+		(property "P/N" "3568"
+			(at 261.62 158.75 90)
 			(effects
 				(font
@@
 			)
 		)
-		(property "Description" "Mounting Hole without connection"
+		(property "Description" ""
 			(at 57.15 176.53 0)
 			(effects
@@
 		)
 		(property "Manufacturer Prt #" ""
+			(at 57.15 176.53 0)
+			(effects
+				(font
+					(size 1.27 1.27)
+				)
+				(hide yes)
+			)
+		)
+		(property "P/N" "~"
 			(at 57.15 176.53 0)
 			(effects
@@
 			)
 		)
-		(property "Description" "Mounting Hole without connection"
+		(property "Description" ""
 			(at 57.15 191.77 0)
 			(effects
@@
 			)
 		)
+		(property "P/N" "~"
+			(at 57.15 191.77 0)
+			(effects
+				(font
+					(size 1.27 1.27)
+				)
+				(hide yes)
+			)
+		)
 		(instances
 			(project "ControlsLeader_PCB"
@@
 			)
 		)
-		(property "Footprint" "Capacitor_SMD:C_0603_1608Metric_Pad1.08x0.95mm_HandSolder"
+		(property "Footprint" "Resistor_SMD:R_0603_1608Metric_Pad0.98x0.95mm_HandSolder"
 			(at 273.05 152.908 90)
 			(effects
@@
 			)
 		)
-		(property "Description" "Resistor"
+		(property "Description" "Controls R47"
 			(at 273.05 151.13 0)
 			(effects
@@
 			)
 		)
+		(property "P/N" "CRCW12101K10FKEAHP"
+			(at 273.05 151.13 90)
+			(effects
+				(font
+					(size 1.27 1.27)
+				)
+				(hide yes)
+			)
+		)
 		(pin "1"
 		)
@@
 			)
 		)
-		(property "Footprint" "Capacitor_SMD:C_0603_1608Metric_Pad1.08x0.95mm_HandSolder"
+		(property "Footprint" "Resistor_SMD:R_0603_1608Metric_Pad0.98x0.95mm_HandSolder"
 			(at 273.05 140.208 90)
 			(effects
@@
 			)
 		)
-		(property "Description" "Resistor"
+		(property "Description" "Controls R47"
 			(at 273.05 138.43 0)
 			(effects
@@
 			)
 		)
+		(property "P/N" "CRCW12101K10FKEAHP"
+			(at 273.05 138.43 90)
+			(effects
+				(font
+					(size 1.27 1.27)
+				)
+				(hide yes)
+			)
+		)
 		(pin "1"
 		)
@@
 			)
 		)
-		(property "Description" "Connector"
+		(property "Description" "Car Can Out"
 			(at 142.24 151.13 0)
 			(effects
@@
 			)
 		)
-		(property "P/N" "1053091102"
+		(property "P/N" "1053131102"
 			(at 142.24 151.13 0)
 			(effects
@@
 			)
 		)
-		(property "Description" "Mounting Hole without connection"
+		(property "Description" ""
 			(at 25.4 191.77 0)
 			(effects
@@
 			)
 		)
+		(property "P/N" "~"
+			(at 25.4 191.77 0)
+			(effects
+				(font
+					(size 1.27 1.27)
+				)
+				(hide yes)
+			)
+		)
 		(instances
 			(project "ControlsLeader_PCB"
@@
 			)
 		)
-		(property "Description" "Generic connector, single row, 01x04, script generated (kicad-library-utils/schlib/autogen/connector/)"
+		(property "Description" "Ign Conn"
 			(at 137.16 31.75 0)
+			(effects
+				(font
+					(size 1.27 1.27)
+				)
+				(hide yes)
+			)
+		)
+		(property "P/N" "1053131104"
+			(at 137.16 31.75 90)
 			(effects
 				(font
@@
 			)
 		)
-		(property "Description" "Connector"
+		(property "Description" "Car Can In"
 			(at 142.24 142.24 0)
 			(effects
@@
 			)
 		)
-		(property "P/N" "1053091102"
+		(property "P/N" "1053131102"
 			(at 142.24 142.24 0)
 			(effects
@@
 			)
 		)
-		(property "Description" "Light emitting diode"
+		(property "Description" "5LDO LED"
 			(at 266.7 142.24 0)
 			(effects
@@
 		)
 		(property "Manufacturer Prt #" "LS Q976.01-N1Q2-1-20-R18"
+			(at 266.7 142.24 0)
+			(effects
+				(font
+					(size 1.27 1.27)
+				)
+				(hide yes)
+			)
+		)
+		(property "P/N" "LS Q976.01-N1Q2-1-20-R18"
 			(at 266.7 142.24 0)
 			(effects
@@
 			)
 		)
-		(property "Description" "Mounting Hole without connection"
+		(property "Description" ""
 			(at 25.4 176.53 0)
 			(effects
@@
 			)
 		)
+		(property "P/N" "~"
+			(at 25.4 176.53 0)
+			(effects
+				(font
+					(size 1.27 1.27)
+				)
+				(hide yes)
+			)
+		)
 		(instances
 			(project "ControlsLeader_PCB"
@@
 			)
 		)
-		(property "Description" "Generic connector, single row, 01x07, script generated (kicad-library-utils/schlib/autogen/connector/)"
+		(property "Description" "Steering Conn"
+			(at 187.96 147.32 0)
+			(effects
+				(font
+					(size 1.27 1.27)
+				)
+				(hide yes)
+			)
+		)
+		(property "P/N" "1053131107"
 			(at 187.96 147.32 0)
 			(effects
@@
 		(unit 2)
 		(exclude_from_sim no)
-		(in_bom yes)
+		(in_bom no)
 		(on_board yes)
 		(dnp no)
@@
 			)
 		)
-		(property "Description" "Symbol for both board-to-board connectors from the LeaderSOM"
+		(property "Description" ""
 			(at 153.924 81.28 0)
 			(effects
@@
 			)
 		)
+		(property "P/N" "~"
+			(at 153.67 90.17 0)
+			(effects
+				(font
+					(size 1.27 1.27)
+				)
+				(hide yes)
+			)
+		)
 		(pin "21"
 		)
@@
 			)
 		)
-		(property "Description" "Connection to the car's Peripheral CAN bus."
+		(property "Description" "PH Can Out"
 			(at 147.32 184.15 0)
 			(effects
@@
 			)
 		)
-		(property "P/N" "105309-1204 "
+		(property "P/N" "1053131104"
 			(at 147.32 184.15 0)
 			(effects
@@
 		(unit 1)
 		(exclude_from_sim no)
-		(in_bom yes)
+		(in_bom no)
 		(on_board yes)
 		(dnp no)
@@
 			)
 		)
-		(property "Description" "Symbol for both board-to-board connectors from the LeaderSOM"
+		(property "Description" ""
 			(at 99.314 81.28 0)
 			(effects
@@
 			(at 99.06 90.17 0)
 			(effects
+				(font
+					(size 1.27 1.27)
+				)
+				(hide yes)
+			)
+		)
+		(property "P/N" "~"
+			(at 99.06 90.17 0)
+			(effects
