File: hardware/ControlsLeader_PCB/Swe_LEDs.kicad_sch (KiCad schematic)
At the start: 14 parts

Commit message: Schematic Ready for Review - Just need FET footprints to be confirmed
Parts:
- D19, D20, D21, D22, D23, D24, D25: footprint (none) -> LED_SMD:LED_0201_0603Metric_Pad0.64x0.40mm_HandSolder
- R48, R49, R50, R51, R52, R53, R54: footprint (none) -> Capacitor_SMD:C_0201_0603Metric_Pad0.64x0.40mm_HandSolder
