File: hardware/ControlsLeader_PCB/24v_5v_buck.kicad_sch (KiCad schematic)
At the start: 13 parts, among them U6 TPS5405DR

Commit message: Final reviews addressed - RevA
Connections:
- net LX: now reaches C31.2, D4.1 (K), L1.1, U6.8 (LX)
