File: hardware/ControlsLeader_PCB/Steering_Wheel.kicad_sch (KiCad schematic)
At the start: 6 parts, among them J10 Indicator_Switch, Q6 NMOS

Commit message: Updated GPIO table, addressed lakshay review
Parts:
- R11: P/N (none) -> CRCW080510K0FKEAC
Changed lines of the file:
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@@
+			)
+		)
+		(property "P/N" "CRCW080510K0FKEAC"
+			(at 187.96 59.69 0)
+			(effects
+				(font
+					(size 1.27 1.27)
+				)
+				(hide yes)
 			)
 		)

Commit message: BOM!
Parts:
- F2: P/N (none) -> 3568
- Horn2, Regen_Active1: now left out of the parts list
- J10: P/N 43650-0300 -> (none); now left out of the parts list
- Q6: P/N (none) -> IRLML2030TRPBF
- R11: footprint Capacitor_SMD:C_0603_1608Metric_Pad1.08x0.95mm_HandSolder -> Resistor_SMD:R_0603_1608Metric_Pad0.98x0.95mm_HandSolder; P/N CRCW080510K0FKEAC -> CRCW060310K0FKTAHP
Changed lines of the file:
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@@
 			)
 		)
-		(property "Footprint" "Capacitor_SMD:C_0603_1608Metric_Pad1.08x0.95mm_HandSolder"
+		(property "Footprint" "Resistor_SMD:R_0603_1608Metric_Pad0.98x0.95mm_HandSolder"
 			(at 186.182 59.69 90)
 			(effects
@@
 			)
 		)
-		(property "Description" "Resistor"
+		(property "Description" "NOMS 10k"
 			(at 187.96 59.69 0)
 			(effects
@@
 			)
 		)
-		(property "P/N" "CRCW080510K0FKEAC"
+		(property "P/N" "CRCW060310K0FKTAHP"
 			(at 187.96 59.69 0)
 			(effects
@@
 		(unit 1)
 		(exclude_from_sim no)
-		(in_bom yes)
+		(in_bom no)
 		(on_board no)
 		(dnp yes)
@@
 			)
 		)
-		(property "Description" "Generic connector, single row, 01x03, script generated (kicad-library-utils/schlib/autogen/connector/)"
+		(property "Description" ""
 			(at 200.66 143.51 0)
 			(effects
@@
 			)
 		)
-		(property "P/N" "43650-0300"
+		(property "P/N" "~"
 			(at 200.66 143.51 0)
 			(effects
@@
 			)
 		)
-		(property "Description" "N-MOSFET transistor, drain/source/gate"
+		(property "Description" "NMOS!"
 			(at 196.85 50.8 0)
 			(effects
@@
 		)
 		(property "Manufacturer Prt #" ""
+			(at 196.85 50.8 0)
+			(effects
+				(font
+					(size 1.27 1.27)
+				)
+				(hide yes)
+			)
+		)
+		(property "P/N" "IRLML2030TRPBF"
 			(at 196.85 50.8 0)
 			(effects
@@
 			)
 		)
-		(property "Description" "Fuse"
+		(property "Description" "Fuse_3.3LDO"
 			(at 205.74 36.83 0)
+			(effects
+				(font
+					(size 1.27 1.27)
+				)
+				(hide yes)
+			)
+		)
+		(property "P/N" "3568"
+			(at 205.74 36.83 90)
 			(effects
 				(font
@@
 		(unit 1)
 		(exclude_from_sim no)
-		(in_bom yes)
+		(in_bom no)
 		(on_board no)
 		(dnp yes)
@@
 			)
 		)
-		(property "Description" "Push button switch, generic, two pins"
+		(property "Description" ""
 			(at 205.74 123.19 0)
 			(effects
@@
 		)
 		(property "Manufacturer Prt #" ""
+			(at 205.74 123.19 0)
+			(effects
+				(font
+					(size 1.27 1.27)
+				)
+				(hide yes)
+			)
+		)
+		(property "P/N" "~"
 			(at 205.74 123.19 0)
 			(effects
@@
 		(unit 1)
 		(exclude_from_sim no)
-		(in_bom yes)
+		(in_bom no)
 		(on_board no)
 		(dnp yes)
@@
 			)
 		)
-		(property "Description" "Push button switch, generic, two pins"
+		(property "Description" ""
 			(at 205.74 105.41 0)
 			(effects
@@
 			(at 205.74 105.41 0)
 			(effects
+				(font
+					(size 1.27 1.27)
+				)
+				(hide yes)
+			)
+		)
+		(property "P/N" "~"
+			(at 205.74 105.41 0)
+			(effects
