File: hardware/ControlsLeader_PCB/dash.kicad_sch (KiCad schematic)
At the start: 10 parts, among them J11 EStop1, J13 Supp_Out, J7 Conn_01x04, J9 Supp_In

Commit message: BOM!
Parts:
- Cruise_Enable1, Cruise_Set1, Gear1, Hazard1, Ignition1, Regen_Enable1: now left out of the parts list
- J11, J13, J9: P/N 43650-0215 -> 1053131102
- J7: P/N (none) -> 1053131104
Changed lines of the file:
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@@
 		(unit 1)
 		(exclude_from_sim no)
-		(in_bom yes)
+		(in_bom no)
 		(on_board no)
 		(dnp yes)
@@
 			)
 		)
-		(property "Description" "Push button switch, generic, two pins"
+		(property "Description" ""
 			(at 242.57 95.25 0)
 			(effects
@@
 		)
 		(property "Manufacturer Prt #" ""
+			(at 242.57 95.25 0)
+			(effects
+				(font
+					(size 1.27 1.27)
+				)
+				(hide yes)
+			)
+		)
+		(property "P/N" "~"
 			(at 242.57 95.25 0)
 			(effects
@@
 			)
 		)
-		(property "Description" "Generic connector, single row, 01x02, script generated (kicad-library-utils/schlib/autogen/connector/)"
+		(property "Description" "EStop_2pin"
 			(at 162.56 140.97 0)
 			(effects
@@
 			)
 		)
-		(property "P/N" "43650-0215"
+		(property "P/N" "1053131102"
 			(at 162.56 140.97 0)
 			(effects
@@
 		(unit 1)
 		(exclude_from_sim no)
-		(in_bom yes)
+		(in_bom no)
 		(on_board no)
 		(dnp yes)
@@
 			)
 		)
-		(property "Description" "Switch, three position, single pole triple throw, 3 position switch, SP3T"
+		(property "Description" ""
 			(at 241.3 72.39 0)
 			(effects
@@
 		)
 		(property "Manufacturer Prt #" ""
+			(at 241.3 72.39 0)
+			(effects
+				(font
+					(size 1.27 1.27)
+				)
+				(hide yes)
+			)
+		)
+		(property "P/N" "~"
 			(at 241.3 72.39 0)
 			(effects
@@
 		(unit 1)
 		(exclude_from_sim no)
-		(in_bom yes)
+		(in_bom no)
 		(on_board no)
 		(dnp yes)
@@
 			)
 		)
-		(property "Description" "Push button switch, generic, two pins"
+		(property "Description" ""
 			(at 242.57 130.81 0)
 			(effects
@@
 		)
 		(property "Manufacturer Prt #" ""
+			(at 242.57 130.81 0)
+			(effects
+				(font
+					(size 1.27 1.27)
+				)
+				(hide yes)
+			)
+		)
+		(property "P/N" "~"
 			(at 242.57 130.81 0)
 			(effects
@@
 			)
 		)
-		(property "Description" "Generic connector, single row, 01x02, script generated (kicad-library-utils/schlib/autogen/connector/)"
+		(property "Description" "Supp IN"
 			(at 134.62 134.62 0)
 			(effects
@@
 			)
 		)
-		(property "P/N" "43650-0215"
+		(property "P/N" "1053131102"
 			(at 134.62 134.62 0)
 			(effects
@@
 			)
 		)
-		(property "Description" "Generic connector, single row, 01x02, script generated (kicad-library-utils/schlib/autogen/connector/)"
+		(property "Description" "Supp OUT"
 			(at 133.35 148.59 0)
 			(effects
@@
 			)
 		)
-		(property "P/N" "43650-0215"
+		(property "P/N" "1053131102"
 			(at 133.35 148.59 0)
 			(effects
@@
 			)
 		)
-		(property "Description" "Generic connector, single row, 01x04, script generated (kicad-library-utils/schlib/autogen/connector/)"
+		(property "Description" "EStop_4pin"
+			(at 195.58 137.16 0)
+			(effects
+				(font
+					(size 1.27 1.27)
+				)
+				(hide yes)
+			)
+		)
+		(property "P/N" "1053131104"
 			(at 195.58 137.16 0)
 			(effects
@@
 		(unit 1)
 		(exclude_from_sim no)
-		(in_bom yes)
+		(in_bom no)
 		(on_board no)
 		(dnp yes)
@@
 			)
 		)
-		(property "Description" "Push button switch, generic, two pins"
+		(property "Description" ""
 			(at 242.57 148.59 0)
 			(effects
@@
 		)
 		(property "Manufacturer Prt #" ""
+			(at 242.57 148.59 0)
+			(effects
+				(font
+					(size 1.27 1.27)
+				)
+				(hide yes)
+			)
+		)
+		(property "P/N" "~"
 			(at 242.57 148.59 0)
 			(effects
@@
 		(unit 1)
 		(exclude_from_sim no)
-		(in_bom yes)
+		(in_bom no)
 		(on_board no)
 		(dnp yes)
@@
 			)
 		)
-		(property "Description" "Push button switch, generic, two pins"
+		(property "Description" ""
 			(at 242.57 111.76 0)
 			(effects
@@
 		)
 		(property "Manufacturer Prt #" ""
+			(at 242.57 111.76 0)
+			(effects
+				(font
+					(size 1.27 1.27)
+				)
+				(hide yes)
+			)
+		)
+		(property "P/N" "~"
 			(at 242.57 111.76 0)
 			(effects
@@
 		(unit 1)
 		(exclude_from_sim no)
-		(in_bom yes)
+		(in_bom no)
 		(on_board no)
 		(dnp yes)
@@
 			)
 		)
-		(property "Description" "Switch, three position, single pole triple throw, 3 position switch, SP3T"
+		(property "Description" ""
 			(at 241.3 54.61 0)
 			(effects
@@
 			(at 241.3 54.61 0)
 			(effects
+				(font
+					(size 1.27 1.27)
+				)
+				(hide yes)
+			)
+		)
+		(property "P/N" "~"
+			(at 241.3 54.61 0)
+			(effects
